Commit message: rename

File: robot_description/urdf/andbot.xacro (robot description, xacro)
@@ -24,11 +24,11 @@
       <origin xyz="0 0 0" rpy="0 0 0"/>
       <geometry>
-        <mesh filename="package://micro_zachbot/robot_description/mesh/head.STL"/>
-      </geometry>
-    </collision>
-    <visual>
-      <origin xyz="0 0 0" rpy="0 0 0"/>
-      <geometry>
-        <mesh filename="package://micro_zachbot/robot_description/mesh/head.STL"/>
+        <mesh filename="package://NextBot/robot_description/mesh/head.STL"/>
+      </geometry>
+    </collision>
+    <visual>
+      <origin xyz="0 0 0" rpy="0 0 0"/>
+      <geometry>
+        <mesh filename="package://NextBot/robot_description/mesh/head.STL"/>
       </geometry>
        <material name="Blue">
@@ -70,11 +70,11 @@
       <origin xyz="0 0 0" rpy="0 0 0"/>
       <geometry>
-        <mesh filename="package://micro_zachbot/robot_description/mesh/fake_body.STL"/>
-      </geometry>
-    </collision>
-    <visual>
-      <origin xyz="0 0 0" rpy="0 0 0"/>
-      <geometry>
-        <mesh filename="package://micro_zachbot/robot_description/mesh/fake_body.STL"/>
+        <mesh filename="package://NextBot/robot_description/mesh/fake_body.STL"/>
+      </geometry>
+    </collision>
+    <visual>
+      <origin xyz="0 0 0" rpy="0 0 0"/>
+      <geometry>
+        <mesh filename="package://NextBot/robot_description/mesh/fake_body.STL"/>
       </geometry>
        <material name="Blue">
@@ -101,5 +101,5 @@
       <origin xyz="0 0 0" rpy="-1.5707 1.5707 0"/>
       <geometry>
-        <mesh filename="package://micro_zachbot/robot_description/mesh/arm_link1.STL"/>
+        <mesh filename="package://NextBot/robot_description/mesh/arm_link1.STL"/>
       </geometry>
     </collision>
@@ -107,5 +107,5 @@
       <origin xyz="0 0 0" rpy="-1.5707 1.5707 0"/>
       <geometry>
-        <mesh filename="package://micro_zachbot/robot_description/mesh/arm_link1.STL"/>
+        <mesh filename="package://NextBot/robot_description/mesh/arm_link1.STL"/>
       </geometry>
        <material name="Blue">
@@ -133,5 +133,5 @@
       <origin xyz="0 0 0" rpy="-1.5707 1.5707 0"/>
       <geometry>
-        <mesh filename="package://micro_zachbot/robot_description/mesh/arm_link2.STL"/>
+        <mesh filename="package://NextBot/robot_description/mesh/arm_link2.STL"/>
       </geometry>
     </collision>
@@ -139,5 +139,5 @@
       <origin xyz="0 0 0" rpy="-1.5707 1.5707 0"/>
       <geometry>
-        <mesh filename="package://micro_zachbot/robot_description/mesh/arm_link2.STL"/>
+        <mesh filename="package://NextBot/robot_description/mesh/arm_link2.STL"/>
       </geometry>
        <material name="Blue">
@@ -165,5 +165,5 @@
       <origin xyz="0 0 0" rpy="1.57 1.5707 0"/>
       <geometry>
-        <mesh filename="package://micro_zachbot/robot_description/mesh/arm_link1.STL"/>
+        <mesh filename="package://NextBot/robot_description/mesh/arm_link1.STL"/>
       </geometry>
     </collision>
@@ -171,5 +171,5 @@
       <origin xyz="0 0 0" rpy="1.57 1.5707 0"/>
       <geometry>
-        <mesh filename="package://micro_zachbot/robot_description/mesh/arm_link1.STL"/>
+        <mesh filename="package://NextBot/robot_description/mesh/arm_link1.STL"/>
       </geometry>
        <material name="Blue">
@@ -197,5 +197,5 @@
       <origin xyz="0 0 0" rpy="-1.5707 1.5707 3.14"/>
       <geometry>
-        <mesh filename="package://micro_zachbot/robot_description/mesh/arm_link2.STL"/>
+        <mesh filename="package://NextBot/robot_description/mesh/arm_link2.STL"/>
       </geometry>
     </collision>
@@ -203,5 +203,5 @@
       <origin xyz="0 0 0" rpy="-1.5707 1.5707 0"/>
       <geometry>
-        <mesh filename="package://micro_zachbot/robot_description/mesh/arm_link2.STL"/>
+        <mesh filename="package://NextBot/robot_description/mesh/arm_link2.STL"/>
       </geometry>
        <material name="Blue">
@@ -229,5 +229,5 @@
       <origin xyz="0 0 ${radius_wheel-height_wheels_from_base}" rpy="0 0 0"/>
       <geometry>
-        <mesh filename="package://micro_zachbot/robot_description/mesh/base_part.STL"/>
+        <mesh filename="package://NextBot/robot_description/mesh/base_part.STL"/>
       </geometry>
     </collision>
@@ -235,5 +235,5 @@
       <origin xyz="0 0 ${radius_wheel-height_wheels_from_base}" rpy="0 0 0"/>
       <geometry>
-        <mesh filename="package://micro_zachbot/robot_description/mesh/base_part.STL"/>
+        <mesh filename="package://NextBot/robot_description/mesh/base_part.STL"/>
       </geometry>
        <material name="Orange">
@@ -254,5 +254,5 @@
       <origin xyz="0 0 -0.019" rpy="1.57 0 -1.57"/>
       <geometry>
-        <mesh filename="package://micro_zachbot/robot_description/mesh/lidar_XV-11.STL"/>
+        <mesh filename="package://NextBot/robot_description/mesh/lidar_XV-11.STL"/>
       </geometry>
     </collision>
@@ -260,5 +260,5 @@
       <origin xyz="0 0 -0.019" rpy="1.57 0 -1.57"/>
       <geometry>
-        <mesh filename="package://micro_zachbot/robot_description/mesh/lidar_XV-11.STL"/>
+        <mesh filename="package://NextBot/robot_description/mesh/lidar_XV-11.STL"/>
       </geometry>
        <material name="Green">
@@ -319,5 +319,5 @@
       <origin xyz="0 0 0" rpy="0 1.570795 1.570795"/>
       <geometry>
-        <mesh filename="package://micro_zachbot/robot_description/mesh/wheel-D152_SMALL.STL"/>
+        <mesh filename="package://NextBot/robot_description/mesh/wheel-D152_SMALL.STL"/>
       </geometry>
     </collision>
@@ -325,5 +325,5 @@
       <origin xyz="0 0 0" rpy="0 1.570795 1.570795"/>
       <geometry>
-        <mesh filename="package://micro_zachbot/robot_description/mesh/wheel-D152_SMALL.STL"/>
+        <mesh filename="package://NextBot/robot_description/mesh/wheel-D152_SMALL.STL"/>
       </geometry>
        <material name="Black">
@@ -370,5 +370,5 @@
       <origin xyz="0 0 0" rpy="0 1.570795 1.570795"/>
       <geometry>
-        <mesh filename="package://micro_zachbot/robot_description/mesh/wheel-D152_SMALL.STL"/>
+        <mesh filename="package://NextBot/robot_description/mesh/wheel-D152_SMALL.STL"/>
       </geometry>
     </collision>
@@ -376,5 +376,5 @@
       <origin xyz="0 0 0" rpy="0 1.570795 1.570795"/>
       <geometry>
-        <mesh filename="package://micro_zachbot/robot_description/mesh/wheel-D152_SMALL.STL"/>
+        <mesh filename="package://NextBot/robot_description/mesh/wheel-D152_SMALL.STL"/>
       </geometry>
        <material name="Black">
